File: BrainPadWiFi.brd (EAGLE design)
At the start: 25.9 x 26.3 mm, 16 parts, among them IC1 ESP-WROOM-02FRONT-FACE, J1 GROVE I2C, U2 TLV1117LV33DCYRDCY4-M

Commit message: Add parts number markers.
Parts:
- removed U$2: (no value), BrainPadWiFi:TWIGLOGO_SMALL
- added U$3: (no value), BrainPadWiFi:OSH-LOGO
Other:
- board text added: "BrainPadWiFi 2.0"
- board text added: "C1"
- board text added: "C2"
- board text added: "C3"
- board text added: "C4"
- board text added: "C5"
- board text added: "I2C 3.3V"
- board text added: "LED1"
- board text added: "LED2"
- board text added: "R1"
- board text added: "R2"
- board text added: "R4"
- board text added: "R5"
- board text added: "U2"
- board text removed: "BrainPadWiFi 1.1"
- board text removed: "STAT1"
Changed lines of the file:
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@@
 <drawing>
 <settings>
-<setting alwaysvectorfont="yes"/>
+<setting alwaysvectorfont="no"/>
 <setting verticaltext="up"/>
 </settings>
-<grid distance="50" unitdist="mil" unit="mil" style="lines" multiple="1" display="no" altdistance="5" altunitdist="mil" altunit="mil"/>
+<grid distance="1" unitdist="mic" unit="mic" style="lines" multiple="1" display="no" altdistance="5" altunitdist="mil" altunit="mil"/>
 <layers>
 <layer number="1" name="Top" color="4" fill="1" visible="yes" active="yes"/>
@@
 <layer number="19" name="Unrouted" color="6" fill="1" visible="yes" active="yes"/>
 <layer number="20" name="Dimension" color="24" fill="1" visible="yes" active="yes"/>
-<layer number="21" name="tPlace" color="7" fill="1" visible="no" active="yes"/>
-<layer number="22" name="bPlace" color="7" fill="1" visible="no" active="yes"/>
+<layer number="21" name="tPlace" color="7" fill="1" visible="yes" active="yes"/>
+<layer number="22" name="bPlace" color="7" fill="1" visible="yes" active="yes"/>
 <layer number="23" name="tOrigins" color="15" fill="1" visible="yes" active="yes"/>
 <layer number="24" name="bOrigins" color="15" fill="1" visible="yes" active="yes"/>
@@
 <layer number="134" name="silk_top" color="7" fill="1" visible="no" active="no"/>
 <layer number="135" name="silk_bottom" color="7" fill="1" visible="no" active="no"/>
-<layer number="136" name="silktop" color="7" fill="1" visible="yes" active="yes"/>
-<layer number="137" name="silkbottom" color="7" fill="1" visible="yes" active="yes"/>
+<layer number="136" name="silktop" color="7" fill="1" visible="no" active="yes"/>
+<layer number="137" name="silkbottom" color="7" fill="1" visible="no" active="yes"/>
 <layer number="144" name="DrillLegend" color="7" fill="1" visible="no" active="no"/>
-<layer number="145" name="DrillLegend_01-16" color="7" fill="1" visible="yes" active="yes"/>
-<layer number="146" name="DrillLegend_01-20" color="7" fill="1" visible="yes" active="yes"/>
+<layer number="145" name="DrillLegend_01-16" color="7" fill="1" visible="no" active="yes"/>
+<layer number="146" name="DrillLegend_01-20" color="7" fill="1" visible="no" active="yes"/>
 <layer number="150" name="Notes" color="7" fill="1" visible="no" active="no"/>
 <layer number="151" name="HeatSink" color="14" fill="1" visible="no" active="no"/>
@@
 <layer number="154" name="FabDoc2" color="2" fill="1" visible="no" active="no"/>
 <layer number="155" name="FabDoc3" color="7" fill="15" visible="no" active="no"/>
-<layer number="166" name="AntennaArea" color="7" fill="1" visible="yes" active="yes"/>
-<layer number="168" name="4mmHeightArea" color="7" fill="1" visible="yes" active="yes"/>
+<layer number="166" name="AntennaArea" color="7" fill="1" visible="no" active="yes"/>
+<layer number="168" name="4mmHeightArea" color="7" fill="1" visible="no" active="yes"/>
 <layer number="199" name="Contour" color="7" fill="1" visible="no" active="no"/>
 <layer number="200" name="200bmp" color="1" fill="10" visible="no" active="no"/>
@@
 <board>
 <plain>
-<text x="3.81" y="21.971" size="1.6764" layer="48" font="vector" ratio="15">BrainPadWiFi 1.1</text>
-<text x="15.367" y="24.765" size="1.016" layer="48" font="vector" ratio="12">STAT1</text>
+<text x="3.81" y="21.971" size="1.6764" layer="48" font="vector" ratio="15">BrainPadWiFi 2.0</text>
 <wire x1="1.016" y1="25.273" x2="24.892" y2="25.273" width="1.2192" layer="48"/>
 <wire x1="24.892" y1="25.273" x2="24.892" y2="3.175" width="1.2192" layer="48"/>
@@
 <wire x1="22.733" y1="1.016" x2="1.016" y2="1.016" width="1.2192" layer="48"/>
 <wire x1="1.016" y1="1.016" x2="1.016" y2="25.273" width="1.2192" layer="48"/>
-<text x="13.462" y="18.542" size="0.8128" layer="48" font="vector" ratio="15">S1  S2</text>
+<text x="13.462" y="18.837" size="0.8128" layer="48" font="vector" ratio="15">S1  S2</text>
+<text x="4.372" y="3.907" size="0.8128" layer="48" font="vector" ratio="15" rot="R90">I2C 3.3V</text>
+<wire x1="17.15" y1="7.025" x2="17.15" y2="2.095" width="0.15" layer="48"/>
+<wire x1="17.15" y1="2.095" x2="19.17" y2="2.095" width="0.15" layer="48"/>
+<wire x1="19.17" y1="2.095" x2="19.17" y2="7.025" width="0.15" layer="48"/>
+<wire x1="19.17" y1="7.025" x2="17.15" y2="7.025" width="0.15" layer="48"/>
+<wire x1="21.825" y1="13.25" x2="19.805" y2="13.25" width="0.15" layer="48"/>
+<wire x1="19.805" y1="13.25" x2="19.805" y2="8.32" width="0.15" layer="48"/>
+<wire x1="19.805" y1="8.32" x2="21.825" y2="8.32" width="0.15" layer="48"/>
+<wire x1="21.825" y1="8.32" x2="21.825" y2="13.25" width="0.15" layer="48"/>
+<wire x1="8.642" y1="18.845" x2="10.662" y2="18.845" width="0.15" layer="48"/>
+<wire x1="10.662" y1="18.845" x2="10.662" y2="13.915" width="0.15" layer="48"/>
+<wire x1="10.662" y1="13.915" x2="8.642" y2="13.915" width="0.15" layer="48"/>
+<wire x1="8.642" y1="13.915" x2="8.642" y2="18.845" width="0.15" layer="48"/>
+<wire x1="11.183" y1="18.846" x2="11.183" y2="13.916" width="0.15" layer="48"/>
+<wire x1="13.203" y1="14.4" x2="13.203" y2="18.846" width="0.15" layer="48"/>
+<wire x1="13.203" y1="18.846" x2="11.183" y2="18.846" width="0.15" layer="48"/>
+<wire x1="17.27" y1="18.849" x2="19.29" y2="18.849" width="0.15" layer="48"/>
+<wire x1="19.29" y1="18.849" x2="19.29" y2="13.919" width="0.15" layer="48"/>
+<wire x1="17.27" y1="14.4" x2="17.27" y2="18.849" width="0.15" layer="48"/>
+<wire x1="19.817" y1="18.851" x2="21.837" y2="18.851" width="0.15" layer="48"/>
+<wire x1="21.837" y1="18.851" x2="21.837" y2="13.921" width="0.15" layer="48"/>
+<wire x1="21.837" y1="13.921" x2="19.817" y2="13.921" width="0.15" layer="48"/>
+<wire x1="19.817" y1="13.921" x2="19.817" y2="18.851" width="0.15" layer="48"/>
+<wire x1="16.328" y1="4.07" x2="16.328" y2="2.05" width="0.15" layer="48"/>
+<wire x1="16.328" y1="2.05" x2="11.418" y2="2.05" width="0.15" layer="48"/>
+<wire x1="11.418" y1="2.05" x2="11.418" y2="4.07" width="0.15" layer="48"/>
+<wire x1="11.418" y1="4.07" x2="16.328" y2="4.07" width="0.15" layer="48"/>
+<wire x1="17.15" y1="7.025" x2="19.17" y2="7.025" width="0.15" layer="48"/>
+<wire x1="19.17" y1="7.025" x2="19.17" y2="2.095" width="0.15" layer="48"/>
+<wire x1="19.17" y1="2.095" x2="17.15" y2="2.095" width="0.15" layer="48"/>
+<wire x1="17.15" y1="2.095" x2="17.15" y2="7.025" width="0.15" layer="48"/>
+<wire x1="20.088" y1="7.024" x2="22.108" y2="7.024" width="0.15" layer="48"/>
+<wire x1="22.108" y1="7.024" x2="22.108" y2="2.094" width="0.15" layer="48"/>
+<wire x1="22.108" y1="2.094" x2="20.088" y2="2.094" width="0.15" layer="48"/>
+<wire x1="20.088" y1="2.094" x2="20.088" y2="7.024" width="0.15" layer="48"/>
+<wire x1="20.53" y1="21.595" x2="20.53" y2="19.84" width="0.15" layer="48"/>
+<wire x1="20.53" y1="19.84" x2="15.311" y2="19.84" width="0.15" layer="48"/>
+<wire x1="15.311" y1="19.84" x2="15.311" y2="21.595" width="0.15" layer="48"/>
+<wire x1="15.311" y1="21.595" x2="20.53" y2="21.595" width="0.15" layer="48"/>
+<wire x1="15.06" y1="21.595" x2="15.06" y2="19.84" width="0.15" layer="48"/>
+<wire x1="15.06" y1="19.84" x2="9.841" y2="19.84" width="0.15" layer="48"/>
+<wire x1="9.841" y1="19.84" x2="9.841" y2="21.595" width="0.15" layer="48"/>
+<wire x1="9.841" y1="21.595" x2="15.06" y2="21.595" width="0.15" layer="48"/>
+<wire x1="16.3" y1="7.1" x2="16.3" y2="5.08" width="0.15" layer="48"/>
+<wire x1="16.3" y1="5.08" x2="11.39" y2="5.08" width="0.15" layer="48"/>
+<wire x1="11.39" y1="5.08" x2="11.39" y2="7.1" width="0.15" layer="48"/>
+<wire x1="11.39" y1="7.1" x2="16.3" y2="7.1" width="0.15" layer="48"/>
+<text x="11.74" y="16.073" size="0.6096" layer="48" font="vector" ratio="15">C5</text>
+<text x="9.175" y="16.072" size="0.6096" layer="48" font="vector" ratio="15">R2</text>
+<text x="17.892" y="16.1" size="0.6096" layer="48" font="vector" ratio="15">R1</text>
+<text x="20.409" y="16.087" size="0.6096" layer="48" font="vector" ratio="15">R4</text>
+<text x="14.774" y="12.111" size="0.6096" layer="48" font="vector" ratio="15">U2</text>
+<text x="20.34" y="10.48" size="0.6096" layer="48" font="vector" ratio="15">R5</text>
+<text x="20.683" y="4.271" size="0.6096" layer="48" font="vector" ratio="15">C4</text>
+<text x="17.759" y="4.271" size="0.6096" layer="48" font="vector" ratio="15">C1</text>
+<text x="14.142" y="5.703" size="0.6096" layer="48" font="vector" ratio="15" rot="R90">C2</text>
+<text x="14.142" y="2.642" size="0.6096" layer="48" font="vector" ratio="15" rot="R90">C3</text>
+<text x="11.521" y="20.403" size="0.6096" layer="48" font="vector" ratio="15">LED1</text>
+<text x="16.976" y="20.394" size="0.6096" layer="48" font="vector" ratio="15">LED2</text>
 </plain>
 <attributes>
@@
 <element name="LED1" library="BrainPadWiFi" package="SML1206" package3d_urn="urn:adsk.eagle:package:15829/1" value="STATUS1" x="12.446" y="20.701"/>
 <element name="J1" library="BrainPadWiFi" package="HW4-2.0" value="GROVE I2C" x="7.366" y="6.096" rot="R270"/>
-<element name="U$2" library="BrainPadWiFi" package="TWIGLOGO_SMALL" value="" x="3.175" y="14.224"/>
+<element name="U$3" library="BrainPadWiFi" package="OSH-LOGO" value="" x="3.715" y="17.678"/>
 </elements>
 <signals>
